File: TS2/v2/page5.sch (KiCad schematic (older format))
At the start: 5 parts

Commit message: more fixup of deleted pages.
Parts:
- removed D2, E2: HM6264, symbol HM6264
- removed D3, E3: 2764, symbol 2764
- removed G1: 74LS04, symbol 74LS04
- added U15, U17: HM6264, symbol HM6264
- added U16, U18: 2764, symbol 2764
Connections:
- net A01: now also U15.10 (A0), U16.10 (A0), U17.10 (A0), U18.10 (A0)
- net A02: now also U15.9 (A1), U16.9 (A1), U17.9 (A1), U18.9 (A1)
- net A03: now also U15.8 (A2), U16.8 (A2), U17.8 (A2), U18.8 (A2)
- net A04: now also U15.7 (A3), U16.7 (A3), U17.7 (A3), U18.7 (A3)
- net A05: now also U15.6 (A4), U16.6 (A4), U17.6 (A4), U18.6 (A4)
- net A06: now also U15.5 (A5), U16.5 (A5), U17.5 (A5), U18.5 (A5)
- net A07: now also U15.4 (A6), U16.4 (A6), U17.4 (A6), U18.4 (A6)
- net A08: now also U15.3 (A7), U16.3 (A7), U17.3 (A7), U18.3 (A7)
- net A09: now also U15.25 (A8), U16.25 (A8), U17.25 (A8), U18.25 (A8)
- net A10: now also U15.24 (A9), U16.24 (A9), U17.24 (A9), U18.24 (A9)
- net A11: now also U15.21 (A10), U16.21 (A10), U17.21 (A10), U18.21 (A10)
- net A12: now also U15.23 (A11), U16.23 (A11), U17.23 (A11), U18.23 (A11)
- net A13: now also U15.2 (A12), U16.2 (A12), U17.2 (A12), U18.2 (A12)
- net D00: now also U15.11 (D0), U16.11 (D0)
- net D01: now also U15.12 (D1), U16.12 (D1)
- net D02: now also U15.13 (D2), U16.13 (D2)
- net D03: now also U15.15 (D3), U16.15 (D3)
- net D04: now also U15.16 (D4), U16.16 (D4)
- net D05: now also U15.17 (D5), U16.17 (D5)
- net D06: now also U15.18 (D6), U16.18 (D6)
- net D07: now also U15.19 (D7), U16.19 (D7)
- net D08: now also U17.11 (D0), U18.11 (D0)
- net D09: now also U17.12 (D1), U18.12 (D1)
- net D10: now also U17.13 (D2), U18.13 (D2)
- net D11: now also U17.15 (D3), U18.15 (D3)
- net D12: now also U17.16 (D4), U18.16 (D4)
- net D13: now also U17.17 (D5), U18.17 (D5)
- net D14: now also U17.18 (D6), U18.18 (D6)
- net D15: now also U17.19 (D7), U18.19 (D7)
- net GND: now also U15.14 (GND), U15.22 (OE), U16.14 (GND), U17.14 (GND), U17.22 (OE), U18.14 (GND)
- net R*/W: now also U16.22 (OE), U18.22 (OE)
- net R/W*: now also U15.27 (WE), U17.27 (WE)
- net VCC: now also U15.26 (CS2), U15.28 (VCC), U16.1 (VPP), U16.27 (~PGM), U16.28 (VCC), U17.26 (CS2), U17.28 (VCC), U18.1 (VPP), U18.27 (~PGM), U18.28 (VCC)
- new net CS_RAM2L*: U15.20 (CS1)
- new net CS_RAM2U*: U17.20 (CS1)
- new net CS_ROM2L*: U16.20 (CE)
- new net CS_ROM2U*: U18.20 (CE)
Changed lines of the file:
@@
 $Descr A 11000 8500
 encoding utf-8
-Sheet 6 8
+Sheet 5 8
 Title "TS2 68000 Single Board Computer"
 Date "2016-09-03"
 Rev "2.0"
 Comp ""
-Comment1 "RAM and ROM (1 of 2)"
+Comment1 "RAM and ROM (2 of 2)"
 Comment2 ""
 Comment3 ""
@@
 $EndDescr
 $Comp
-L 2764 D3
-U 1 1 57C37A1F
+L 2764 U16
+U 1 1 57CAE145
 P 4350 5100
-F 0 "D3" H 4100 6100 50  0000 C CNN
+F 0 "U16" H 4100 6100 50  0000 C CNN
 F 1 "2764" H 4350 4100 50  0000 C CNN
 F 2 "" H 4350 5100 50  0000 C CNN
@@
 $EndComp
 $Comp
-L 2764 E3
-U 1 1 57C37AB5
+L 2764 U18
+U 1 1 57CAE146
 P 7600 5100
-F 0 "E3" H 7350 6100 50  0000 C CNN
+F 0 "U18" H 7350 6100 50  0000 C CNN
 F 1 "2764" H 7600 4100 50  0000 C CNN
 F 2 "" H 7600 5100 50  0000 C CNN
@@
 $EndComp
 $Comp
-L HM6264 D2
-U 1 1 57CAE143
+L HM6264 U15
+U 1 1 57C33086
 P 4350 2450
-F 0 "D2" H 4100 3450 50  0000 C CNN
+F 0 "U15" H 4100 3450 50  0000 C CNN
 F 1 "HM6264" H 4350 1450 50  0000 C CNN
 F 2 "" H 4350 2450 50  0000 C CNN
@@
 $EndComp
 $Comp
-L HM6264 E2
-U 1 1 57CAE144
+L HM6264 U17
+U 1 1 57C330E4
 P 7600 2450
-F 0 "E2" H 7350 3450 50  0000 C CNN
+F 0 "U17" H 7350 3450 50  0000 C CNN
 F 1 "HM6264" H 7600 1450 50  0000 C CNN
 F 2 "" H 7600 2450 50  0000 C CNN
@@
 	1    0    0    -1
 $EndComp
-$Comp
-L 74LS04 G1
-U 3 1 57C33190
-P 3000 3950
-F 0 "G1" H 3195 4065 50  0000 C CNN
-F 1 "74LS04" H 3190 3825 50  0000 C CNN
-F 2 "" H 3000 3950 50  0000 C CNN
-F 3 "" H 3000 3950 50  0000 C CNN
-	3    3000 3950
-	1    0    0    -1
-$EndComp
-Wire Wire Line
-	2550 3650 2550 3950
 Wire Wire Line
 	2300 3650 6900 3650
 Wire Wire Line
 	3650 3650 3650 3300
-Connection ~ 2550 3650
 Text GLabel 2300 3650 0    60   Input ~ 0
 R/W*
@@
 	3650 3150 2300 3150
 Text GLabel 2300 3150 0    60   Input ~ 0
-CS_RAM1L*
-Wire Wire Line
-	3450 3750 3450 6000
+CS_RAM2L*
+Wire Wire Line
+	3450 3950 3450 6000
 Wire Wire Line
 	2300 1550 3650 1550
@@
 	5050 1650 5350 1650
 $Comp
-L GND #PWR021
-U 1 1 57CAE147
+L GND #PWR35
+U 1 1 57C4A627
 P 5050 3250
-F 0 "#PWR021" H 5050 3000 50  0001 C CNN
+F 0 "#PWR35" H 5050 3000 50  0001 C CNN
 F 1 "GND" H 5050 3100 50  0000 C CNN
 F 2 "" H 5050 3250 50  0000 C CNN
@@
 $EndComp
 $Comp
-L VCC #PWR022
-U 1 1 57CAE148
+L VCC #PWR34
+U 1 1 57C4A645
 P 5050 3150
-F 0 "#PWR022" H 5050 3000 50  0001 C CNN
+F 0 "#PWR34" H 5050 3000 50  0001 C CNN
 F 1 "VCC" H 5050 3300 50  0000 C CNN
 F 2 "" H 5050 3150 50  0000 C CNN
@@
 $EndComp
 $Comp
-L VCC #PWR023
-U 1 1 57CAE149
+L VCC #PWR41
+U 1 1 57C4A66D
 P 8300 3150
-F 0 "#PWR023" H 8300 3000 50  0001 C CNN
+F 0 "#PWR41" H 8300 3000 50  0001 C CNN
 F 1 "VCC" H 8300 3300 50  0000 C CNN
 F 2 "" H 8300 3150 50  0000 C CNN
@@
 $EndComp
 $Comp
-L GND #PWR024
-U 1 1 57CAE14A
+L GND #PWR42
+U 1 1 57C4A68B
 P 8300 3250
-F 0 "#PWR024" H 8300 3000 50  0001 C CNN
+F 0 "#PWR42" H 8300 3000 50  0001 C CNN
 F 1 "GND" H 8300 3100 50  0000 C CNN
 F 2 "" H 8300 3250 50  0000 C CNN
@@
 A01
 $Comp
-L VCC #PWR025
-U 1 1 57CAE14B
+L VCC #PWR30
+U 1 1 57C4B0B4
 P 4350 1500
-F 0 "#PWR025" H 4350 1350 50  0001 C CNN
+F 0 "#PWR30" H 4350 1350 50  0001 C CNN
 F 1 "VCC" H 4350 1650 50  0000 C CNN
 F 2 "" H 4350 1500 50  0000 C CNN
@@
 $EndComp
 $Comp
-L GND #PWR026
-U 1 1 57CAE14C
+L GND #PWR31
+U 1 1 57C4B0FA
 P 4350 3400
-F 0 "#PWR026" H 4350 3150 50  0001 C CNN
+F 0 "#PWR31" H 4350 3150 50  0001 C CNN
 F 1 "GND" H 4350 3250 50  0000 C CNN
 F 2 "" H 4350 3400 50  0000 C CNN
@@
 	2300 4300 3650 4300
 Text GLabel 2300 5900 0    60   Input ~ 0
-CS_ROM1L*
-$Comp
-L GND #PWR027
-U 1 1 57CAE14D
+CS_ROM2L*
+$Comp
+L GND #PWR33
+U 1 1 57C52013
 P 4350 6050
-F 0 "#PWR027" H 4350 5800 50  0001 C CNN
+F 0 "#PWR33" H 4350 5800 50  0001 C CNN
 F 1 "GND" H 4350 5900 50  0000 C CNN
 F 2 "" H 4350 6050 50  0000 C CNN
@@
 $EndComp
 $Comp
-L VCC #PWR028
-U 1 1 57C52031
+L VCC #PWR32
+U 1 1 57CAE14E
 P 4350 4150
-F 0 "#PWR028" H 4350 4000 50  0001 C CNN
+F 0 "#PWR32" H 4350 4000 50  0001 C CNN
 F 1 "VCC" H 4350 4300 50  0000 C CNN
 F 2 "" H 4350 4150 50  0000 C CNN
@@
 	3550 5700 3550 5600
 $Comp
-L VCC #PWR029
-U 1 1 57C5238F
+L VCC #PWR29
+U 1 1 57CAE14F
 P 3300 5600
-F 0 "#PWR029" H 3300 5450 50  0001 C CNN
+F 0 "#PWR29" H 3300 5450 50  0001 C CNN
 F 1 "VCC" H 3300 5750 50  0000 C CNN
 F 2 "" H 3300 5600 50  0000 C CNN
@@
 Connection ~ 3650 3650
 $Comp
-L VCC #PWR030
-U 1 1 57C5501D
+L VCC #PWR37
+U 1 1 57CAE150
 P 7600 1500
-F 0 "#PWR030" H 7600 1350 50  0001 C CNN
+F 0 "#PWR37" H 7600 1350 50  0001 C CNN
 F 1 "VCC" H 7600 1650 50  0000 C CNN
 F 2 "" H 7600 1500 50  0000 C CNN
@@
 $EndComp
 $Comp
-L GND #PWR031
-U 1 1 57C5503B
+L GND #PWR38
+U 1 1 57CAE151
 P 7600 3400
-F 0 "#PWR031" H 7600 3150 50  0001 C CNN
+F 0 "#PWR38" H 7600 3150 50  0001 C CNN
 F 1 "GND" H 7600 3250 50  0000 C CNN
 F 2 "" H 7600 3400 50  0000 C CNN
@@
 $EndComp
 Text GLabel 6450 3150 0    60   Input ~ 0
-CS_RAM1U*
+CS_RAM2U*
 Wire Wire Line
 	6450 3150 6900 3150
@@
 	6450 4200 6900 4200
 $Comp
-L VCC #PWR032
-U 1 1 57C5736B
+L VCC #PWR39
+U 1 1 57CAE152
 P 7600 4150
-F 0 "#PWR032" H 7600 4000 50  0001 C CNN
+F 0 "#PWR39" H 7600 4000 50  0001 C CNN
 F 1 "VCC" H 7600 4300 50  0000 C CNN
 F 2 "" H 7600 4150 50  0000 C CNN
@@
 $EndComp
 $Comp
-L GND #PWR033
-U 1 1 57C573B1
+L GND #PWR40
+U 1 1 57CAE153
 P 7600 6050
-F 0 "#PWR033" H 7600 5800 50  0001 C CNN
+F 0 "#PWR40" H 7600 5800 50  0001 C CNN
 F 1 "GND" H 7600 5900 50  0000 C CNN
 F 2 "" H 7600 6050 50  0000 C CNN
@@
 Connection ~ 6800 5600
 $Comp
-L VCC #PWR034
-U 1 1 57CAE154
+L VCC #PWR36
+U 1 1 57C575E7
 P 6500 5600
-F 0 "#PWR034" H 6500 5450 50  0001 C CNN
+F 0 "#PWR36" H 6500 5450 50  0001 C CNN
 F 1 "VCC" H 6500 5750 50  0000 C CNN
 F 2 "" H 6500 5600 50  0000 C CNN
@@
 	6450 4300 6900 4300
 Text GLabel 6450 5900 0    60   Input ~ 0
-CS_ROM1U*
+CS_ROM2U*
 Wire Wire Line
 	6450 5900 6900 5900
 Wire Wire Line
-	3450 3950 6700 3950
+	2300 3950 6700 3950
 Wire Wire Line
 	6700 3950 6700 6000
 Wire Wire Line
 	6700 6000 6900 6000
-Text GLabel 2300 3950 0    60   Output ~ 0
+Connection ~ 3450 3950
+Text GLabel 2300 3950 0    60   Input ~ 0
 R*/W
-Wire Wire Line
-	2300 3950 2400 3950
-Wire Wire Line
-	2400 3950 2400 3750
-Wire Wire Line
-	2400 3750 3450 3750
-Connection ~ 3450 3950
 $EndSCHEMATC
