File: TS2/v2/page5.sch (KiCad schematic (older format))
At the start: 4 parts, among them U15 HM6264, U16 28C64, U17 HM6264, U18 28C64

Commit message: Add all bypass caps, show pullups as SIP resistors, start PCB layout.
Parts:
- U15, U16, U17, U18: footprint (none) -> Housings_DIP:DIP-28_W7.62mm
Changed lines of the file:
@@
 Sheet 6 9
 Title "TS2 68000 Single Board Computer"
-Date "2017-01-19"
+Date "2017-01-23"
 Rev "2.0"
 Comp "Jeff Tranter"
@@
 F 0 "U15" H 4350 2600 50  0000 C CNN
 F 1 "HM6264" H 4350 2450 50  0000 C CNN
-F 2 "" H 4350 2450 50  0000 C CNN
+F 2 "Housings_DIP:DIP-28_W7.62mm" H 4350 2450 50  0001 C CNN
 F 3 "" H 4350 2450 50  0000 C CNN
 	1    4350 2450
@@
 F 0 "U17" H 7600 2600 50  0000 C CNN
 F 1 "HM6264" H 7600 2450 50  0000 C CNN
-F 2 "" H 7600 2450 50  0000 C CNN
+F 2 "Housings_DIP:DIP-28_W7.62mm" H 7600 2450 50  0001 C CNN
 F 3 "" H 7600 2450 50  0000 C CNN
 	1    7600 2450
@@
 	5050 1650 5350 1650
 $Comp
-L GND #PWR056
+L GND #PWR058
 U 1 1 57C4A627
 P 5050 3250
-F 0 "#PWR056" H 5050 3000 50  0001 C CNN
+F 0 "#PWR058" H 5050 3000 50  0001 C CNN
 F 1 "GND" H 5050 3100 50  0000 C CNN
 F 2 "" H 5050 3250 50  0000 C CNN
@@
 $EndComp
 $Comp
-L VCC #PWR057
+L VCC #PWR059
 U 1 1 57C4A645
 P 5050 3150
-F 0 "#PWR057" H 5050 3000 50  0001 C CNN
+F 0 "#PWR059" H 5050 3000 50  0001 C CNN
 F 1 "VCC" H 5050 3300 50  0000 C CNN
 F 2 "" H 5050 3150 50  0000 C CNN
@@
 $EndComp
 $Comp
-L VCC #PWR058
+L VCC #PWR060
 U 1 1 57C4A66D
 P 8300 3150
-F 0 "#PWR058" H 8300 3000 50  0001 C CNN
+F 0 "#PWR060" H 8300 3000 50  0001 C CNN
 F 1 "VCC" H 8300 3300 50  0000 C CNN
 F 2 "" H 8300 3150 50  0000 C CNN
@@
 $EndComp
 $Comp
-L GND #PWR059
+L GND #PWR061
 U 1 1 57C4A68B
 P 8300 3250
-F 0 "#PWR059" H 8300 3000 50  0001 C CNN
+F 0 "#PWR061" H 8300 3000 50  0001 C CNN
 F 1 "GND" H 8300 3100 50  0000 C CNN
 F 2 "" H 8300 3250 50  0000 C CNN
@@
 A01
 $Comp
-L VCC #PWR060
+L VCC #PWR062
 U 1 1 57C4B0B4
 P 4350 1500
-F 0 "#PWR060" H 4350 1350 50  0001 C CNN
+F 0 "#PWR062" H 4350 1350 50  0001 C CNN
 F 1 "VCC" H 4350 1650 50  0000 C CNN
 F 2 "" H 4350 1500 50  0000 C CNN
@@
 $EndComp
 $Comp
-L GND #PWR061
+L GND #PWR063
 U 1 1 57C4B0FA
 P 4350 3400
-F 0 "#PWR061" H 4350 3150 50  0001 C CNN
+F 0 "#PWR063" H 4350 3150 50  0001 C CNN
 F 1 "GND" H 4350 3250 50  0000 C CNN
 F 2 "" H 4350 3400 50  0000 C CNN
@@
 CS_ROM2L*
 $Comp
-L GND #PWR062
+L GND #PWR064
 U 1 1 57C52013
 P 4350 6050
-F 0 "#PWR062" H 4350 5800 50  0001 C CNN
+F 0 "#PWR064" H 4350 5800 50  0001 C CNN
 F 1 "GND" H 4350 5900 50  0000 C CNN
 F 2 "" H 4350 6050 50  0000 C CNN
@@
 $EndComp
 $Comp
-L VCC #PWR063
+L VCC #PWR065
 U 1 1 57CAE14E
 P 4350 4150
-F 0 "#PWR063" H 4350 4000 50  0001 C CNN
+F 0 "#PWR065" H 4350 4000 50  0001 C CNN
 F 1 "VCC" H 4350 4300 50  0000 C CNN
 F 2 "" H 4350 4150 50  0000 C CNN
@@
 	3300 5600 3650 5600
 $Comp
-L VCC #PWR064
+L VCC #PWR066
 U 1 1 57CAE14F
 P 3300 5600
-F 0 "#PWR064" H 3300 5450 50  0001 C CNN
+F 0 "#PWR066" H 3300 5450 50  0001 C CNN
 F 1 "VCC" H 3300 5750 50  0000 C CNN
 F 2 "" H 3300 5600 50  0000 C CNN
@@
 Connection ~ 3650 3650
 $Comp
-L VCC #PWR065
+L VCC #PWR067
 U 1 1 57CAE150
 P 7600 1500
-F 0 "#PWR065" H 7600 1350 50  0001 C CNN
+F 0 "#PWR067" H 7600 1350 50  0001 C CNN
 F 1 "VCC" H 7600 1650 50  0000 C CNN
 F 2 "" H 7600 1500 50  0000 C CNN
@@
 $EndComp
 $Comp
-L GND #PWR066
+L GND #PWR068
 U 1 1 57CAE151
 P 7600 3400
-F 0 "#PWR066" H 7600 3150 50  0001 C CNN
+F 0 "#PWR068" H 7600 3150 50  0001 C CNN
 F 1 "GND" H 7600 3250 50  0000 C CNN
 F 2 "" H 7600 3400 50  0000 C CNN
@@
 	6450 4200 6900 4200
 $Comp
-L VCC #PWR067
+L VCC #PWR069
 U 1 1 57CAE152
 P 7600 4150
-F 0 "#PWR067" H 7600 4000 50  0001 C CNN
+F 0 "#PWR069" H 7600 4000 50  0001 C CNN
 F 1 "VCC" H 7600 4300 50  0000 C CNN
 F 2 "" H 7600 4150 50  0000 C CNN
@@
 $EndComp
 $Comp
-L GND #PWR068
+L GND #PWR070
 U 1 1 57CAE153
 P 7600 6050
-F 0 "#PWR068" H 7600 5800 50  0001 C CNN
+F 0 "#PWR070" H 7600 5800 50  0001 C CNN
 F 1 "GND" H 7600 5900 50  0000 C CNN
 F 2 "" H 7600 6050 50  0000 C CNN
@@
 Connection ~ 6800 5600
 $Comp
-L VCC #PWR069
+L VCC #PWR071
 U 1 1 57C575E7
 P 6500 5600
-F 0 "#PWR069" H 6500 5450 50  0001 C CNN
+F 0 "#PWR071" H 6500 5450 50  0001 C CNN
 F 1 "VCC" H 6500 5750 50  0000 C CNN
 F 2 "" H 6500 5600 50  0000 C CNN
@@
 F 0 "U16" H 4350 5250 50  0000 C CNN
 F 1 "28C64" H 4350 5100 50  0000 C CNN
-F 2 "" H 4350 5100 50  0000 C CNN
+F 2 "Housings_DIP:DIP-28_W7.62mm" H 4350 5100 50  0001 C CNN
 F 3 "" H 4350 5100 50  0000 C CNN
 	1    4350 5100
@@
 F 0 "U18" H 7600 5250 50  0000 C CNN
 F 1 "28C64" H 7600 5100 50  0000 C CNN
-F 2 "" H 7600 5100 50  0000 C CNN
+F 2 "Housings_DIP:DIP-28_W7.62mm" H 7600 5100 50  0001 C CNN
 F 3 "" H 7600 5100 50  0000 C CNN
 	1    7600 5100
