File: TS2/v2/page2.sch (KiCad schematic (older format))
At the start: 6 parts, among them U10 74LS32, U19 74LS20, U24 74LS260, U25 74LS260, U26 74LS138, U27 25LS2548

Commit message: Add all bypass caps, show pullups as SIP resistors, start PCB layout.
Parts:
- U10, U19, U24, U25: footprint (none) -> Housings_DIP:DIP-14_W7.62mm
- U26: footprint ~ -> Housings_DIP:DIP-16_W7.62mm
- U27: footprint (none) -> Housings_DIP:DIP-20_W7.62mm
Changed lines of the file:
@@
 Sheet 3 9
 Title "TS2 68000 Single Board Computer"
-Date "2017-01-19"
+Date "2017-01-23"
 Rev "2.0"
 Comp "Jeff Tranter"
@@
 F 0 "U26" H 7900 1900 60  0000 C CNN
 F 1 "74LS138" H 7850 1750 60  0000 C CNN
-F 2 "~" H 7900 1750 60  0000 C CNN
+F 2 "Housings_DIP:DIP-16_W7.62mm" H 7900 1750 60  0001 C CNN
 F 3 "~" H 7900 1750 60  0000 C CNN
 	1    7900 1750
@@
 F 0 "U10" H 2500 5050 50  0000 C CNN
 F 1 "74LS32" H 2500 4950 50  0000 C CNN
-F 2 "" H 2500 5000 50  0000 C CNN
+F 2 "Housings_DIP:DIP-14_W7.62mm" H 2500 5000 50  0001 C CNN
 F 3 "" H 2500 5000 50  0000 C CNN
 	3    2500 5000
@@
 F 0 "U19" H 6500 5450 50  0000 C CNN
 F 1 "74LS20" H 6500 5250 50  0000 C CNN
-F 2 "" H 6500 5350 50  0000 C CNN
+F 2 "Housings_DIP:DIP-14_W7.62mm" H 6500 5350 50  0001 C CNN
 F 3 "" H 6500 5350 50  0000 C CNN
 	2    6500 5350
@@
 F 0 "U24" H 2800 1250 50  0000 C CNN
 F 1 "74LS260" H 2800 1150 50  0000 C CNN
-F 2 "" H 2800 1200 50  0000 C CNN
+F 2 "Housings_DIP:DIP-14_W7.62mm" H 2800 1200 50  0001 C CNN
 F 3 "" H 2800 1200 50  0000 C CNN
 	1    2800 1200
@@
 F 0 "U25" H 4200 2750 50  0000 C CNN
 F 1 "74LS260" H 4200 2650 50  0000 C CNN
-F 2 "" H 4200 2700 50  0000 C CNN
+F 2 "Housings_DIP:DIP-14_W7.62mm" H 4200 2700 50  0001 C CNN
 F 3 "" H 4200 2700 50  0000 C CNN
 	1    4200 2700
@@
 F 0 "U24" H 2800 3450 50  0000 C CNN
 F 1 "74LS260" H 2800 3350 50  0000 C CNN
-F 2 "" H 2800 3400 50  0000 C CNN
+F 2 "Housings_DIP:DIP-14_W7.62mm" H 2800 3400 50  0001 C CNN
 F 3 "" H 2800 3400 50  0000 C CNN
 	2    2800 3400
@@
 F 0 "U25" H 4200 4550 50  0000 C CNN
 F 1 "74LS260" H 4200 4450 50  0000 C CNN
-F 2 "" H 4200 4500 50  0000 C CNN
+F 2 "Housings_DIP:DIP-14_W7.62mm" H 4200 4500 50  0001 C CNN
 F 3 "" H 4200 4500 50  0000 C CNN
 	2    4200 4500
@@
 F 0 "U27" H 7900 4200 50  0000 C CNN
 F 1 "25LS2548" H 7900 4100 50  0000 C CNN
-F 2 "" H 7900 4100 50  0000 C CNN
+F 2 "Housings_DIP:DIP-20_W7.62mm" H 7900 4100 50  0001 C CNN
 F 3 "" H 7900 4100 50  0000 C CNN
 	1    7900 4100
@@
 NoConn ~ 8500 2100
 $Comp
-L GND #PWR037
+L GND #PWR039
 U 1 1 57C1E00A
 P 7900 2200
-F 0 "#PWR037" H 7900 1950 50  0001 C CNN
+F 0 "#PWR039" H 7900 1950 50  0001 C CNN
 F 1 "GND" H 7900 2050 50  0000 C CNN
 F 2 "" H 7900 2200 50  0000 C CNN
@@
 $EndComp
 $Comp
-L VCC #PWR038
+L VCC #PWR040
 U 1 1 57C1E030
 P 7900 1300
-F 0 "#PWR038" H 7900 1150 50  0001 C CNN
+F 0 "#PWR040" H 7900 1150 50  0001 C CNN
 F 1 "VCC" H 7900 1450 50  0000 C CNN
 F 2 "" H 7900 1300 50  0000 C CNN
@@
 NoConn ~ 8500 4450
 $Comp
-L GND #PWR039
+L GND #PWR041
 U 1 1 57C1E717
 P 8000 4550
-F 0 "#PWR039" H 8000 4300 50  0001 C CNN
+F 0 "#PWR041" H 8000 4300 50  0001 C CNN
 F 1 "GND" H 8000 4400 50  0000 C CNN
 F 2 "" H 8000 4550 50  0000 C CNN
@@
 $EndComp
 $Comp
-L VCC #PWR040
+L VCC #PWR042
 U 1 1 57C1E73D
 P 7900 3650
-F 0 "#PWR040" H 7900 3500 50  0001 C CNN
+F 0 "#PWR042" H 7900 3500 50  0001 C CNN
 F 1 "VCC" H 7900 3800 50  0000 C CNN
 F 2 "" H 7900 3650 50  0000 C CNN
@@
 	7200 3900 7200 3700
 $Comp
-L VCC #PWR041
+L VCC #PWR043
 U 1 1 57C1EB1C
 P 7200 3700
-F 0 "#PWR041" H 7200 3550 50  0001 C CNN
+F 0 "#PWR043" H 7200 3550 50  0001 C CNN
 F 1 "VCC" H 7200 3850 50  0000 C CNN
 F 2 "" H 7200 3700 50  0000 C CNN
