File: TS2/v2/page3.sch (KiCad schematic (older format))
At the start: 5 parts, among them U10 74LS32, U5 74LS04, U7 74LS08, U8 74LS32, U9 74LS32

Commit message: Add all bypass caps, show pullups as SIP resistors, start PCB layout.
Parts:
- U10, U5, U7, U8, U9: footprint (none) -> Housings_DIP:DIP-14_W7.62mm
Changed lines of the file:
@@
 Sheet 4 9
 Title "TS2 68000 Single Board Computer"
-Date "2017-01-19"
+Date "2017-01-23"
 Rev "2.0"
 Comp "Jeff Tranter"
@@
 F 0 "U7" H 4250 3400 50  0000 C CNN
 F 1 "74LS08" H 4250 3300 50  0000 C CNN
-F 2 "" H 4250 3350 50  0000 C CNN
+F 2 "Housings_DIP:DIP-14_W7.62mm" H 4250 3350 50  0001 C CNN
 F 3 "" H 4250 3350 50  0000 C CNN
 	1    4250 3350
@@
 F 0 "U8" H 4250 4850 50  0000 C CNN
 F 1 "74LS32" H 4250 4750 50  0000 C CNN
-F 2 "" H 4250 4800 50  0000 C CNN
+F 2 "Housings_DIP:DIP-14_W7.62mm" H 4250 4800 50  0001 C CNN
 F 3 "" H 4250 4800 50  0000 C CNN
 	1    4250 4800
@@
 F 0 "U8" H 7400 2350 50  0000 C CNN
 F 1 "74LS32" H 7400 2250 50  0000 C CNN
-F 2 "" H 7400 2300 50  0000 C CNN
+F 2 "Housings_DIP:DIP-14_W7.62mm" H 7400 2300 50  0001 C CNN
 F 3 "" H 7400 2300 50  0000 C CNN
 	3    7400 2300
@@
 F 0 "U8" H 7400 2950 50  0000 C CNN
 F 1 "74LS32" H 7400 2850 50  0000 C CNN
-F 2 "" H 7400 2900 50  0000 C CNN
+F 2 "Housings_DIP:DIP-14_W7.62mm" H 7400 2900 50  0001 C CNN
 F 3 "" H 7400 2900 50  0000 C CNN
 	4    7400 2900
@@
 F 0 "U9" H 7400 3550 50  0000 C CNN
 F 1 "74LS32" H 7400 3450 50  0000 C CNN
-F 2 "" H 7400 3500 50  0000 C CNN
+F 2 "Housings_DIP:DIP-14_W7.62mm" H 7400 3500 50  0001 C CNN
 F 3 "" H 7400 3500 50  0000 C CNN
 	1    7400 3500
@@
 F 0 "U9" H 7400 4150 50  0000 C CNN
 F 1 "74LS32" H 7400 4050 50  0000 C CNN
-F 2 "" H 7400 4100 50  0000 C CNN
+F 2 "Housings_DIP:DIP-14_W7.62mm" H 7400 4100 50  0001 C CNN
 F 3 "" H 7400 4100 50  0000 C CNN
 	2    7400 4100
@@
 F 0 "U9" H 7400 4750 50  0000 C CNN
 F 1 "74LS32" H 7400 4650 50  0000 C CNN
-F 2 "" H 7400 4700 50  0000 C CNN
+F 2 "Housings_DIP:DIP-14_W7.62mm" H 7400 4700 50  0001 C CNN
 F 3 "" H 7400 4700 50  0000 C CNN
 	3    7400 4700
@@
 F 0 "U9" H 7400 5350 50  0000 C CNN
 F 1 "74LS32" H 7400 5250 50  0000 C CNN
-F 2 "" H 7400 5300 50  0000 C CNN
+F 2 "Housings_DIP:DIP-14_W7.62mm" H 7400 5300 50  0001 C CNN
 F 3 "" H 7400 5300 50  0000 C CNN
 	4    7400 5300
@@
 F 0 "U10" H 7400 5950 50  0000 C CNN
 F 1 "74LS32" H 7400 5850 50  0000 C CNN
-F 2 "" H 7400 5900 50  0000 C CNN
+F 2 "Housings_DIP:DIP-14_W7.62mm" H 7400 5900 50  0001 C CNN
 F 3 "" H 7400 5900 50  0000 C CNN
 	1    7400 5900
@@
 F 0 "U8" H 7400 1750 50  0000 C CNN
 F 1 "74LS32" H 7400 1650 50  0000 C CNN
-F 2 "" H 7400 1700 50  0000 C CNN
+F 2 "Housings_DIP:DIP-14_W7.62mm" H 7400 1700 50  0001 C CNN
 F 3 "" H 7400 1700 50  0000 C CNN
 	2    7400 1700
@@
 F 0 "U5" H 3445 4365 50  0000 C CNN
 F 1 "74LS04" H 3440 4125 50  0000 C CNN
-F 2 "" H 3250 4250 50  0000 C CNN
+F 2 "Housings_DIP:DIP-14_W7.62mm" H 3250 4250 50  0001 C CNN
 F 3 "" H 3250 4250 50  0000 C CNN
 	3    3250 4250
