File: TS2/v2/page4.sch (KiCad schematic (older format))
At the start: 5 parts, among them U11 HM6264, U12 28C64, U13 HM6264, U14 28C64, U5 74LS04

Commit message: Add all bypass caps, show pullups as SIP resistors, start PCB layout.
Parts:
- U11, U12, U13, U14: footprint (none) -> Housings_DIP:DIP-28_W7.62mm
- U5: footprint (none) -> Housings_DIP:DIP-14_W7.62mm
Changed lines of the file:
@@
 Sheet 5 9
 Title "TS2 68000 Single Board Computer"
-Date "2017-01-19"
+Date "2017-01-23"
 Rev "2.0"
 Comp "Jeff Tranter"
@@
 F 0 "U11" H 4350 2600 50  0000 C CNN
 F 1 "HM6264" H 4350 2450 50  0000 C CNN
-F 2 "" H 4350 2450 50  0000 C CNN
+F 2 "Housings_DIP:DIP-28_W7.62mm" H 4350 2450 50  0001 C CNN
 F 3 "" H 4350 2450 50  0000 C CNN
 	1    4350 2450
@@
 F 0 "U13" H 7600 2600 50  0000 C CNN
 F 1 "HM6264" H 7600 2450 50  0000 C CNN
-F 2 "" H 7600 2450 50  0000 C CNN
+F 2 "Housings_DIP:DIP-28_W7.62mm" H 7600 2450 50  0001 C CNN
 F 3 "" H 7600 2450 50  0000 C CNN
 	1    7600 2450
@@
 F 0 "U5" H 3195 4065 50  0000 C CNN
 F 1 "74LS04" H 3190 3825 50  0000 C CNN
-F 2 "" H 3000 3950 50  0000 C CNN
+F 2 "Housings_DIP:DIP-14_W7.62mm" H 3000 3950 50  0001 C CNN
 F 3 "" H 3000 3950 50  0000 C CNN
 	4    3000 3950
@@
 	5050 1650 5350 1650
 $Comp
-L GND #PWR042
+L GND #PWR044
 U 1 1 57CAE147
 P 5050 3250
-F 0 "#PWR042" H 5050 3000 50  0001 C CNN
+F 0 "#PWR044" H 5050 3000 50  0001 C CNN
 F 1 "GND" H 5050 3100 50  0000 C CNN
 F 2 "" H 5050 3250 50  0000 C CNN
@@
 $EndComp
 $Comp
-L VCC #PWR043
+L VCC #PWR045
 U 1 1 57CAE148
 P 5050 3150
-F 0 "#PWR043" H 5050 3000 50  0001 C CNN
+F 0 "#PWR045" H 5050 3000 50  0001 C CNN
 F 1 "VCC" H 5050 3300 50  0000 C CNN
 F 2 "" H 5050 3150 50  0000 C CNN
@@
 $EndComp
 $Comp
-L VCC #PWR044
+L VCC #PWR046
 U 1 1 57CAE149
 P 8300 3150
-F 0 "#PWR044" H 8300 3000 50  0001 C CNN
+F 0 "#PWR046" H 8300 3000 50  0001 C CNN
 F 1 "VCC" H 8300 3300 50  0000 C CNN
 F 2 "" H 8300 3150 50  0000 C CNN
@@
 $EndComp
 $Comp
-L GND #PWR045
+L GND #PWR047
 U 1 1 57CAE14A
 P 8300 3250
-F 0 "#PWR045" H 8300 3000 50  0001 C CNN
+F 0 "#PWR047" H 8300 3000 50  0001 C CNN
 F 1 "GND" H 8300 3100 50  0000 C CNN
 F 2 "" H 8300 3250 50  0000 C CNN
@@
 A01
 $Comp
-L VCC #PWR046
+L VCC #PWR048
 U 1 1 57CAE14B
 P 4350 1500
-F 0 "#PWR046" H 4350 1350 50  0001 C CNN
+F 0 "#PWR048" H 4350 1350 50  0001 C CNN
 F 1 "VCC" H 4350 1650 50  0000 C CNN
 F 2 "" H 4350 1500 50  0000 C CNN
@@
 $EndComp
 $Comp
-L GND #PWR047
+L GND #PWR049
 U 1 1 57CAE14C
 P 4350 3400
-F 0 "#PWR047" H 4350 3150 50  0001 C CNN
+F 0 "#PWR049" H 4350 3150 50  0001 C CNN
 F 1 "GND" H 4350 3250 50  0000 C CNN
 F 2 "" H 4350 3400 50  0000 C CNN
@@
 CS_ROM1L*
 $Comp
-L GND #PWR048
+L GND #PWR050
 U 1 1 57CAE14D
 P 4350 6050
-F 0 "#PWR048" H 4350 5800 50  0001 C CNN
+F 0 "#PWR050" H 4350 5800 50  0001 C CNN
 F 1 "GND" H 4350 5900 50  0000 C CNN
 F 2 "" H 4350 6050 50  0000 C CNN
@@
 $EndComp
 $Comp
-L VCC #PWR049
+L VCC #PWR051
 U 1 1 57C52031
 P 4350 4150
-F 0 "#PWR049" H 4350 4000 50  0001 C CNN
+F 0 "#PWR051" H 4350 4000 50  0001 C CNN
 F 1 "VCC" H 4350 4300 50  0000 C CNN
 F 2 "" H 4350 4150 50  0000 C CNN
@@
 	3300 5600 3650 5600
 $Comp
-L VCC #PWR050
+L VCC #PWR052
 U 1 1 57C5238F
 P 3300 5600
-F 0 "#PWR050" H 3300 5450 50  0001 C CNN
+F 0 "#PWR052" H 3300 5450 50  0001 C CNN
 F 1 "VCC" H 3300 5750 50  0000 C CNN
 F 2 "" H 3300 5600 50  0000 C CNN
@@
 Connection ~ 3650 3650
 $Comp
-L VCC #PWR051
+L VCC #PWR053
 U 1 1 57C5501D
 P 7600 1500
-F 0 "#PWR051" H 7600 1350 50  0001 C CNN
+F 0 "#PWR053" H 7600 1350 50  0001 C CNN
 F 1 "VCC" H 7600 1650 50  0000 C CNN
 F 2 "" H 7600 1500 50  0000 C CNN
@@
 $EndComp
 $Comp
-L GND #PWR052
+L GND #PWR054
 U 1 1 57C5503B
 P 7600 3400
-F 0 "#PWR052" H 7600 3150 50  0001 C CNN
+F 0 "#PWR054" H 7600 3150 50  0001 C CNN
 F 1 "GND" H 7600 3250 50  0000 C CNN
 F 2 "" H 7600 3400 50  0000 C CNN
@@
 	6450 4200 6900 4200
 $Comp
-L VCC #PWR053
+L VCC #PWR055
 U 1 1 57C5736B
 P 7600 4150
-F 0 "#PWR053" H 7600 4000 50  0001 C CNN
+F 0 "#PWR055" H 7600 4000 50  0001 C CNN
 F 1 "VCC" H 7600 4300 50  0000 C CNN
 F 2 "" H 7600 4150 50  0000 C CNN
@@
 $EndComp
 $Comp
-L GND #PWR054
+L GND #PWR056
 U 1 1 57C573B1
 P 7600 6050
-F 0 "#PWR054" H 7600 5800 50  0001 C CNN
+F 0 "#PWR056" H 7600 5800 50  0001 C CNN
 F 1 "GND" H 7600 5900 50  0000 C CNN
 F 2 "" H 7600 6050 50  0000 C CNN
@@
 Connection ~ 6800 5600
 $Comp
-L VCC #PWR055
+L VCC #PWR057
 U 1 1 57CAE154
 P 6500 5600
-F 0 "#PWR055" H 6500 5450 50  0001 C CNN
+F 0 "#PWR057" H 6500 5450 50  0001 C CNN
 F 1 "VCC" H 6500 5750 50  0000 C CNN
 F 2 "" H 6500 5600 50  0000 C CNN
@@
 F 0 "U12" H 4350 5250 50  0000 C CNN
 F 1 "28C64" H 4350 5100 50  0000 C CNN
-F 2 "" H 4350 5100 50  0000 C CNN
+F 2 "Housings_DIP:DIP-28_W7.62mm" H 4350 5100 50  0001 C CNN
 F 3 "" H 4350 5100 50  0000 C CNN
 	1    4350 5100
@@
 F 0 "U14" H 7600 5250 50  0000 C CNN
 F 1 "28C64" H 7600 5100 50  0000 C CNN
-F 2 "" H 7600 5100 50  0000 C CNN
+F 2 "Housings_DIP:DIP-28_W7.62mm" H 7600 5100 50  0001 C CNN
 F 3 "" H 7600 5100 50  0000 C CNN
 	1    7600 5100
