File: TS2/v2/ts2.kicad_pcb (KiCad board)
At the start: 2 copper layers, 100 parts, among them P1 FTDI (TERMINAL), P2 FTDI (HOST), P3 +5V POWER, SW1 RESET, SW2 SINGLE STEP/RUN, SW3 STEP, SW4 ABORT, SW5 POWER, U1 555, U10 74LS32, U11 HM6264, U12 28C64, U13 HM6264, U14 28C64, U15 HM6264, U16 28C64, U17 HM6264, U18 28C64, U19 74LS20, U2 8 MHz, U20 74LS74, U21 74LS161, U22 74LS161, U23 74LS74, U24 74LS260, U25 74LS260, U26 74LS138, U27 25LS2548, U28 74LS148, U29 6850, U3 74LS00, U30 6850, U31 MC14411, U32 74LS138, U33 74LS138, U34 74LS00, U35 74LS74, U4 74LS06, U5 74LS04, U6 68000, U7 74LS08, U8 74LS32, U9 74LS32, Y1 1.842MHz

Commit message: More work on layout.
Parts:
- moved U27 269.0 mm to (27.9, 167.0)
- moved U7 216.9 mm to (40.6, 109.9)
- moved U8 200.3 mm to (41.3, 133.3)
- moved C3 197.3 mm to (27.9, 153.0)
- moved U9 193.2 mm to (38.1, 178.4)
- moved C1 187.7 mm to (35.6, 158.8)
- moved R1 187.2 mm to (47.6, 157.5)
- moved U25 186.8 mm to (53.3, 108.6)
- moved U24 186.1 mm to (67.9, 109.9)
- moved R4 185.5 mm to (27.3, 146.7)
- moved C2 180.7 mm to (29.8, 158.1), turned to 0 degrees
- moved C25 179.0 mm to (198.1, 18.4)
- moved U1 176.3 mm to (27.3, 134.0)
- moved U32 171.1 mm to (111.8, 68.6)
- moved U10 171.1 mm to (48.3, 177.2)
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
Commit message: More work on layout.
Parts:
- moved RR2 26.6 mm to (82.8, 166.6), turned to 0 degrees
- moved C2 17.3 mm to (45.2, 166.1)
- moved SW3 16.1 mm to (33.3, 213.5)
- moved SW2 15.5 mm to (42.2, 213.5)
- moved R1 15.3 mm to (59.9, 166.6)
- moved R25 14.9 mm to (73.9, 207.1)
- moved D1 14.9 mm to (58.7, 213.5)
- moved SW1 14.9 mm to (51.1, 213.5)
- moved U34 14.8 mm to (113.7, 116.2)
- moved D2 14.2 mm to (73.9, 213.5)
- moved SW4 14.2 mm to (81.5, 213.5)
- moved SW5 14.2 mm to (66.3, 213.5)
- moved C3 13.6 mm to (27.9, 166.6)
- moved U11 11.6 mm to (31.0, 31.5)
- moved JP1 11.2 mm to (78.7, 142.7)
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
Commit message: Working on PCB layout.
Parts:
- JP1, JP2, JP3, JP4, JP5, JP6: footprint Buttons_Switches_ThroughHole:SW_DIP_x1_Slide -> Connect:PINHEAD1-2
- U11, U12, U13, U14, U15, U16, U17, U18: footprint Housings_DIP:DIP-28_W7.62mm -> Housings_DIP:DIP-28_W15.24mm
- U29, U30, U31: footprint Housings_DIP:DIP-24_W7.62mm -> Housings_DIP:DIP-24_W15.24mm
- U6: footprint Housings_DIP:DIP-64_W15.24mm -> Housings_DIP:DIP-64_W22.86mm
- moved C25 213.0 mm to (30.5, 149.9)
- moved C33 185.1 mm to (55.9, 180.3)
- moved C32 182.3 mm to (43.2, 180.3)
- moved C37 179.9 mm to (106.7, 180.3)
- moved C11 166.6 mm to (33.0, 78.7)
- moved C28 165.8 mm to (68.6, 149.9)
- moved C35 163.9 mm to (81.3, 180.3)
- moved C18 157.6 mm to (43.2, 121.9)
- moved C31 144.8 mm to (30.5, 180.3)
- moved C30 142.9 mm to (121.9, 160.0)
- moved C12 140.9 mm to (53.3, 78.7)
- moved C34 140.4 mm to (68.6, 180.3)
- moved C26 136.3 mm to (43.2, 149.9)
- moved C20 131.4 mm to (68.6, 121.9)
- moved C24 125.3 mm to (106.7, 121.9)
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Other:
- board text added: "TS2 Single Board Computer Rev 2.0 Copyright (c) 2017 Jeff Tranter <tranter@pobox.com>"

Commit message: Working on PCB layout.
Parts:
- added HOLE1: MountingHole_3mm, Mounting_Holes:MountingHole_3mm, F.Cu at (30.5, 22.9)
- added HOLE2: MountingHole_3mm, Mounting_Holes:MountingHole_3mm, F.Cu at (142.2, 22.9)
- added HOLE3: MountingHole_3mm, Mounting_Holes:MountingHole_3mm, F.Cu at (27.9, 228.6)
- added HOLE4: MountingHole_3mm, Mounting_Holes:MountingHole_3mm, F.Cu at (141.0, 229.9)
- moved RR1 10.9 mm to (91.4, 24.1)
- moved C10 10.2 mm to (132.1, 22.9)
- moved U28 10.2 mm to (127.0, 20.3)
- moved D2 8.89 mm to (90.2, 228.6)
- moved R25 8.89 mm to (92.7, 221.0)
- moved SW1 8.89 mm to (59.7, 228.6)
- moved SW2 8.89 mm to (49.5, 228.6)
- moved SW4 8.89 mm to (100.3, 228.6)
- moved SW5 8.89 mm to (80.0, 228.6)
- moved SW3 8.89 mm to (39.4, 228.6)
- moved D1 8.89 mm to (69.8, 228.6)
- moved R6 8.89 mm to (69.8, 221.0)
- moved C4 7.62 mm to (61.0, 22.9)
- moved P3 7.62 mm to (71.1, 22.9)
- moved D3 5.08 mm to (43.2, 22.9)
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Changed lines of the file:
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@@
     (links 625)
     (no_connects 625)
-    (area 24.665 16.783095 149.134049 233.825001)
+    (area 21.451474 16.783095 150.730046 235.84626)
     (thickness 1.6)
     (drawings 1)
     (tracks 0)
     (zones 0)
-    (modules 100)
+    (modules 104)
     (nets 209)
   )
@@
     (0 F.Cu signal)
     (31 B.Cu signal)
-    (33 F.Adhes user hide)
-    (35 F.Paste user hide)
+    (33 F.Adhes user)
+    (35 F.Paste user)
     (37 F.SilkS user)
     (39 F.Mask user)
@@
     (uvia_drill 0.1)
     (uvias_allowed no)
-    (uvia_min_size 0.2)
-    (uvia_min_drill 0.1)
+    (uvia_min_size 0)
+    (uvia_min_drill 0)
     (pcb_text_width 0.3)
     (pcb_text_size 1.5 1.5)
@@
   )
   (module Capacitors_ThroughHole:C_Radial_D5_L6_P2.5 (layer F.Cu)
-    (at 68.58 22.86 180)
+    (at 60.96 22.86 180)
     (descr "Radial Electrolytic Capacitor Diameter 5mm x Length 6mm, Pitch 2.5mm")
     (tags "Electrolytic Capacitor")
@@
   )
   (module Capacitors_ThroughHole:C_Disc_D3_P2.5 (layer F.Cu)
-    (at 35.56 33.02)
+    (at 33.02 33.02)
     (descr "Capacitor 3mm Disc, Pitch 2.5mm")
     (tags Capacitor)
@@
   )
   (module Capacitors_ThroughHole:C_Disc_D3_P2.5 (layer F.Cu)
-    (at 142.24 22.86 270)
+    (at 132.08 22.86 270)
     (descr "Capacitor 3mm Disc, Pitch 2.5mm")
     (tags Capacitor)
@@
   )
   (module Connect:PINHEAD1-2 (layer F.Cu)
-    (at 60.96 228.6)
+    (at 69.85 228.6)
     (attr virtual)
     (fp_text reference D1 (at 0 -3.9) (layer F.SilkS)
@@
   )
   (module Connect:PINHEAD1-2 (layer F.Cu)
-    (at 81.28 228.6)
+    (at 90.17 228.6)
     (attr virtual)
     (fp_text reference D2 (at 0 -3.9) (layer F.SilkS)
@@
   )
   (module Diodes_ThroughHole:Diode_DO-35_SOD27_Horizontal_RM10 (layer F.Cu)
-    (at 48.26 22.86)
+    (at 43.18 22.86)
     (descr "Diode, DO-35,  SOD27, Horizontal, RM 10mm")
     (tags "Diode, DO-35, SOD27, Horizontal, RM 10mm, 1N4148,")
@@
   )
   (module Connect:PINHEAD1-2 (layer F.Cu)
-    (at 78.74 22.86)
+    (at 71.12 22.86)
     (attr virtual)
     (fp_text reference P3 (at 0 -3.9) (layer F.SilkS)
@@
   )
   (module Resistors_ThroughHole:Resistor_Horizontal_RM7mm (layer F.Cu)
-    (at 60.96 220.98)
+    (at 69.85 220.98)
     (descr "Resistor, Axial,  RM 7.62mm, 1/3W,")
     (tags "Resistor Axial RM 7.62mm 1/3W R3")
@@
   )
   (module Resistors_ThroughHole:Resistor_Horizontal_RM7mm (layer F.Cu)
-    (at 83.82 220.98)
+    (at 92.71 220.98)
     (descr "Resistor, Axial,  RM 7.62mm, 1/3W,")
     (tags "Resistor Axial RM 7.62mm 1/3W R3")
@@
   )
   (module Resistors_ThroughHole:Resistor_Array_SIP8 (layer F.Cu)
-    (at 101.6 27.94)
+    (at 91.44 24.13)
     (descr "8 R pack")
     (tags R)
@@
   )
   (module Connect:PINHEAD1-3 (layer F.Cu)
-    (at 50.8 228.6)
+    (at 59.69 228.6)
     (attr virtual)
     (fp_text reference SW1 (at 0.05 -3.8) (layer F.SilkS)
@@
   )
   (module Connect:PINHEAD1-3 (layer F.Cu)
-    (at 40.64 228.6)
+    (at 49.53 228.6)
     (attr virtual)
     (fp_text reference SW2 (at 0.05 -3.8) (layer F.SilkS)
@@
   )
   (module Connect:PINHEAD1-3 (layer F.Cu)
-    (at 30.48 228.6)
+    (at 39.37 228.6)
     (attr virtual)
     (fp_text reference SW3 (at 0.05 -3.8) (layer F.SilkS)
@@
   )
   (module Connect:PINHEAD1-3 (layer F.Cu)
-    (at 91.44 228.6)
+    (at 100.33 228.6)
     (attr virtual)
     (fp_text reference SW4 (at 0.05 -3.8) (layer F.SilkS)
@@
   )
   (module Connect:PINHEAD1-3 (layer F.Cu)
-    (at 71.12 228.6)
+    (at 80.01 228.6)
     (attr virtual)
     (fp_text reference SW5 (at 0.05 -3.8) (layer F.SilkS)
@@
   )
   (module Housings_DIP:DIP-16_W7.62mm (layer F.Cu)
-    (at 137.16 20.32 270)
+    (at 127 20.32 270)
     (descr "16-lead dip package, row spacing 7.62 mm (300 mils)")
     (tags "dil dip 2.54 300")
@@
   )
   (module Crystals:Crystal_HC49-U_Vertical (layer F.Cu)
-    (at 139.7 205.74 270)
+    (at 139.7 205.74 90)
     (descr "Crystal, Quarz, HC49/U, vertical, stehend,")
     (tags "Crystal, Quarz, HC49/U, vertical, stehend,")
-    (fp_text reference Y1 (at 0 -3.81 270) (layer F.SilkS)
+    (fp_text reference Y1 (at 0 -3.81 90) (layer F.SilkS)
       (effects (font (size 1 1) (thickness 0.15)))
     )
-    (fp_text value 1.842MHz (at 0 -4.064 270) (layer F.Fab)
+    (fp_text value 1.842MHz (at 0 -4.064 90) (layer F.Fab)
       (effects (font (size 1 1) (thickness 0.15)))
     )
@@
     (fp_line (start 3.6703 2.29108) (end 4.16052 2.1209) (layer F.SilkS) (width 0.15))
     (fp_line (start -3.2004 -2.32918) (end 3.2512 -2.32918) (layer F.SilkS) (width 0.15))
-    (pad 1 thru_hole circle (at -2.44094 0 270) (size 1.50114 1.50114) (drill 0.8001) (layers *.Cu *.Mask F.SilkS)
+    (pad 1 thru_hole circle (at -2.44094 0 90) (size 1.50114 1.50114) (drill 0.8001) (layers *.Cu *.Mask F.SilkS)
       (net 26 "Net-(R20-Pad2)"))
-    (pad 2 thru_hole circle (at 2.44094 0 270) (size 1.50114 1.50114) (drill 0.8001) (layers *.Cu *.Mask F.SilkS)
+    (pad 2 thru_hole circle (at 2.44094 0 90) (size 1.50114 1.50114) (drill 0.8001) (layers *.Cu *.Mask F.SilkS)
       (net 25 "Net-(R20-Pad1)"))
   )
@@
   )
   (module Connect:PINHEAD1-2 (layer F.Cu)
-    (at 142.24 160.02)
+    (at 142.24 162.56)
     (attr virtual)
     (fp_text reference JP5 (at 0 -3.9) (layer F.SilkS)
@@
       (net 14 "Net-(JP6-Pad2)"))
   )
+  (module Mounting_Holes:MountingHole_3mm (layer F.Cu)
+    (at 30.48 22.86)
+    (descr "Mounting hole, Befestigungsbohrung, 3mm, No Annular, Kein Restring,")
+    (tags "Mounting hole, Befestigungsbohrung, 3mm, No Annular, Kein Restring,")
+    (fp_text reference HOLE1 (at 0 -4.0005) (layer F.SilkS)
+      (effects (font (size 1 1) (thickness 0.15)))
+    )
+    (fp_text value MountingHole_3mm (at 1.00076 5.00126) (layer F.Fab)
+      (effects (font (size 1 1) (thickness 0.15)))
+    )
+    (fp_circle (center 0 0) (end 3 0) (layer Cmts.User) (width 0.381))
+    (pad 1 thru_hole circle (at 0 0) (size 3 3) (drill 3) (layers))
+  )
+  (module Mounting_Holes:MountingHole_3mm (layer F.Cu)
+    (at 142.24 22.86)
+    (descr "Mounting hole, Befestigungsbohrung, 3mm, No Annular, Kein Restring,")
+    (tags "Mounting hole, Befestigungsbohrung, 3mm, No Annular, Kein Restring,")
+    (fp_text reference HOLE2 (at 0 -4.0005) (layer F.SilkS)
+      (effects (font (size 1 1) (thickness 0.15)))
+    )
+    (fp_text value MountingHole_3mm (at 1.00076 5.00126) (layer F.Fab)
+      (effects (font (size 1 1) (thickness 0.15)))
+    )
+    (fp_circle (center 0 0) (end 3 0) (layer Cmts.User) (width 0.381))
+    (pad 1 thru_hole circle (at 0 0) (size 3 3) (drill 3) (layers))
+  )
+  (module Mounting_Holes:MountingHole_3mm (layer F.Cu)
+    (at 140.97 229.87)
+    (descr "Mounting hole, Befestigungsbohrung, 3mm, No Annular, Kein Restring,")
+    (tags "Mounting hole, Befestigungsbohrung, 3mm, No Annular, Kein Restring,")
+    (fp_text reference HOLE4 (at 0 -4.0005) (layer F.SilkS)
+      (effects (font (size 1 1) (thickness 0.15)))
+    )
+    (fp_text value MountingHole_3mm (at 1.00076 5.00126) (layer F.Fab)
+      (effects (font (size 1 1) (thickness 0.15)))
+    )
+    (fp_circle (center 0 0) (end 3 0) (layer Cmts.User) (width 0.381))
+    (pad 1 thru_hole circle (at 0 0) (size 3 3) (drill 3) (layers))
+  )
+  (module Mounting_Holes:MountingHole_3mm (layer F.Cu)
+    (at 27.94 228.6)
+    (descr "Mounting hole, Befestigungsbohrung, 3mm, No Annular, Kein Restring,")
+    (tags "Mounting hole, Befestigungsbohrung, 3mm, No Annular, Kein Restring,")
+    (fp_text reference HOLE3 (at 0 -4.0005) (layer F.SilkS)
+      (effects (font (size 1 1) (thickness 0.15)))
+    )
+    (fp_text value MountingHole_3mm (at 1.00076 5.00126) (layer F.Fab)
+      (effects (font (size 1 1) (thickness 0.15)))
+    )
+    (fp_circle (center 0 0) (end 3 0) (layer Cmts.User) (width 0.381))
+    (pad 1 thru_hole circle (at 0 0) (size 3 3) (drill 3) (layers))
+  )
   (gr_text "TS2 Single Board Computer Rev 2.0\nCopyright (c) 2017\nJeff Tranter <tranter@pobox.com>" (at 78.74 210.82) (layer F.SilkS)

Commit message: Working on PCB layout.
Parts:
- moved HOLE3 2.54 mm to (30.5, 228.6)
- moved HOLE4 1.80 mm to (142.2, 228.6)
Other:
- board outline added: 127 x 221 mm
- board text added: "ABORT"
- board text added: "GND +5V"
- board text added: "HALT"
- board text added: "POWER"
- board text added: "RESET"
- board text added: "STEP"
- board text added: "STEP/RUN"
Changed lines of the file:
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@@
     (links 625)
     (no_connects 625)
-    (area 21.451474 16.783095 150.730046 235.84626)
+    (area 22.784999 15.164999 150.730046 236.295001)
     (thickness 1.6)
-    (drawings 1)
+    (drawings 13)
     (tracks 0)
     (zones 0)
@@
     (descr "Capacitor 3mm Disc, Pitch 2.5mm")
     (tags Capacitor)
-    (fp_text reference C1 (at 2.286 0.508) (layer F.SilkS)
+    (fp_text reference C1 (at 1.27 -2.54) (layer F.SilkS)
       (effects (font (size 1 1) (thickness 0.15)))
     )
@@
     (descr "Capacitor 3mm Disc, Pitch 2.5mm")
     (tags Capacitor)
-    (fp_text reference C2 (at 1.25 -2.5) (layer F.SilkS)
+    (fp_text reference C2 (at 1.27 -2.54) (layer F.SilkS)
       (effects (font (size 1 1) (thickness 0.15)))
     )
@@
     (descr "Capacitor 12mm Disc, Pitch 7.75mm")
     (tags Capacitor)
-    (fp_text reference C3 (at 3.875 -3.5) (layer F.SilkS)
+    (fp_text reference C3 (at 3.81 3.81) (layer F.SilkS)
       (effects (font (size 1 1) (thickness 0.15)))
     )
@@
     (descr "Capacitor 3mm Disc, Pitch 2.5mm")
     (tags Capacitor)
-    (fp_text reference C10 (at 1.25 -2.5 270) (layer F.SilkS)
+    (fp_text reference C10 (at -2.54 0 360) (layer F.SilkS)
       (effects (font (size 1 1) (thickness 0.15)))
     )
-    (fp_text value 0.1uF (at 6.096 0 270) (layer F.Fab)
+    (fp_text value 0.1uF (at 5.08 0 360) (layer F.Fab)
       (effects (font (size 1 1) (thickness 0.15)))
     )
@@
     (at 71.12 22.86)
     (attr virtual)
-    (fp_text reference P3 (at 0 -3.9) (layer F.SilkS)
+    (fp_text reference P3 (at 0 5.08) (layer F.SilkS)
       (effects (font (size 1 1) (thickness 0.15)))
     )
@@
     (descr "Resistor, Axial,  RM 7.62mm, 1/3W,")
     (tags "Resistor Axial RM 7.62mm 1/3W R3")
-    (fp_text reference R1 (at 4.05892 -3.50012 180) (layer F.SilkS)
+    (fp_text reference R1 (at 3.81 2.54 180) (layer F.SilkS)
       (effects (font (size 1 1) (thickness 0.15)))
     )
@@
     (descr "Resistor, Axial,  RM 7.62mm, 1/3W,")
     (tags "Resistor Axial RM 7.62mm 1/3W R3")
-    (fp_text reference R4 (at 4.05892 -3.50012) (layer F.SilkS)
+    (fp_text reference R4 (at 3.81 -2.54) (layer F.SilkS)
       (effects (font (size 1 1) (thickness 0.15)))
     )
@@
       (effects (font (size 1 1) (thickness 0.15)))
     )
-    (fp_text value 4.7K (at 0 2.032) (layer F.Fab)
+    (fp_text value 4.7K (at 0 3.81) (layer F.Fab)
       (effects (font (size 1 1) (thickness 0.15)))
     )
@@
     (descr "8 R pack")
     (tags R)
-    (fp_text reference RR2 (at -1.27 -2.794 270) (layer F.SilkS)
+    (fp_text reference RR2 (at -12.7 0 360) (layer F.SilkS)
       (effects (font (size 1 1) (thickness 0.15)))
     )
@@
     (descr "8 R pack")
     (tags R)
-    (fp_text reference RR3 (at -1.27 -2.794 270) (layer F.SilkS)
+    (fp_text reference RR3 (at -12.7 0 360) (layer F.SilkS)
       (effects (font (size 1 1) (thickness 0.15)))
     )
@@
     (descr "8 R pack")
     (tags R)
-    (fp_text reference RR4 (at -1.27 -2.794 270) (layer F.SilkS)
+    (fp_text reference RR4 (at -12.7 0 360) (layer F.SilkS)
       (effects (font (size 1 1) (thickness 0.15)))
     )
@@
     (descr "16-lead dip package, row spacing 7.62 mm (300 mils)")
     (tags "dil dip 2.54 300")
-    (fp_text reference U28 (at 0 -5.22 270) (layer F.SilkS)
+    (fp_text reference U28 (at -2.54 12.7 360) (layer F.SilkS)
       (effects (font (size 1 1) (thickness 0.15)))
     )
-    (fp_text value 74LS148 (at 0 -3.72 270) (layer F.Fab)
+    (fp_text value 74LS148 (at -2.54 7.62 360) (layer F.Fab)
       (effects (font (size 1 1) (thickness 0.15)))
     )
@@
     (descr "Mounting hole, Befestigungsbohrung, 3mm, No Annular, Kein Restring,")
     (tags "Mounting hole, Befestigungsbohrung, 3mm, No Annular, Kein Restring,")
-    (fp_text reference HOLE1 (at 0 -4.0005) (layer F.SilkS)
+    (fp_text reference HOLE1 (at 0 -4.0005) (layer F.SilkS) hide
       (effects (font (size 1 1) (thickness 0.15)))
     )
@@
     (descr "Mounting hole, Befestigungsbohrung, 3mm, No Annular, Kein Restring,")
     (tags "Mounting hole, Befestigungsbohrung, 3mm, No Annular, Kein Restring,")
-    (fp_text reference HOLE2 (at 0 -4.0005) (layer F.SilkS)
+    (fp_text reference HOLE2 (at 0 -4.0005) (layer F.SilkS) hide
       (effects (font (size 1 1) (thickness 0.15)))
     )
@@
   )
   (module Mounting_Holes:MountingHole_3mm (layer F.Cu)
-    (at 140.97 229.87)
+    (at 142.24 228.6)
     (descr "Mounting hole, Befestigungsbohrung, 3mm, No Annular, Kein Restring,")
     (tags "Mounting hole, Befestigungsbohrung, 3mm, No Annular, Kein Restring,")
-    (fp_text reference HOLE4 (at 0 -4.0005) (layer F.SilkS)
+    (fp_text reference HOLE4 (at 0 -4.0005) (layer F.SilkS) hide
       (effects (font (size 1 1) (thickness 0.15)))
     )
@@
   )
   (module Mounting_Holes:MountingHole_3mm (layer F.Cu)
-    (at 27.94 228.6)
+    (at 30.48 228.6)
     (descr "Mounting hole, Befestigungsbohrung, 3mm, No Annular, Kein Restring,")
     (tags "Mounting hole, Befestigungsbohrung, 3mm, No Annular, Kein Restring,")
-    (fp_text reference HOLE3 (at 0 -4.0005) (layer F.SilkS)
+    (fp_text reference HOLE3 (at 0 -4.0005) (layer F.SilkS) hide
       (effects (font (size 1 1) (thickness 0.15)))
     )
@@
     (pad 1 thru_hole circle (at 0 0) (size 3 3) (drill 3) (layers))
   )
+  (gr_text POWER (at 80.01 233.68) (layer F.SilkS)
+    (effects (font (size 1.5 1.5) (thickness 0.3)))
+  )
+  (gr_text POWER (at 90.17 233.68) (layer F.SilkS)
+    (effects (font (size 1.5 1.5) (thickness 0.3)))
+  )
+  (gr_text ABORT (at 100.33 233.68) (layer F.SilkS)
+    (effects (font (size 1.5 1.5) (thickness 0.3)))
+  )
+  (gr_text HALT (at 69.85 233.68) (layer F.SilkS)
+    (effects (font (size 1.5 1.5) (thickness 0.3)))
+  )
+  (gr_text RESET (at 59.69 233.68) (layer F.SilkS)
+    (effects (font (size 1.5 1.5) (thickness 0.3)))
+  )
+  (gr_text STEP/RUN (at 49.53 233.68) (layer F.SilkS)
+    (effects (font (size 1.5 1.5) (thickness 0.3)))
+  )
+  (gr_text STEP (at 39.37 233.68) (layer F.SilkS)
+    (effects (font (size 1.5 1.5) (thickness 0.3)))
+  )
+  (gr_text "GND +5V" (at 71.12 17.78) (layer F.SilkS)
+    (effects (font (size 1.5 1.5) (thickness 0.3)))
+  )
+  (gr_line (start 22.86 236.22) (end 22.86 15.24) (angle 90) (layer Edge.Cuts) (width 0.15))
+  (gr_line (start 149.86 236.22) (end 22.86 236.22) (angle 90) (layer Edge.Cuts) (width 0.15))
+  (gr_line (start 149.86 15.24) (end 149.86 236.22) (angle 90) (layer Edge.Cuts) (width 0.15))
+  (gr_line (start 22.86 15.24) (end 149.86 15.24) (angle 90) (layer Edge.Cuts) (width 0.15))
   (gr_text "TS2 Single Board Computer Rev 2.0\nCopyright (c) 2017\nJeff Tranter <tranter@pobox.com>" (at 78.74 210.82) (layer F.SilkS)
     (effects (font (size 1.5 1.5) (thickness 0.3)))

Commit message: Initial PCB routing.
Routing:
- net GND: track 0.00 -> 1448.8 mm, vias 0 -> 23
- net VCC: track 0.00 -> 1344.8 mm, vias 0 -> 15
- net A07: track 0.00 -> 427.9 mm, vias 0 -> 5
- net A06: track 0.00 -> 421.2 mm, vias 0 -> 6
- net A03: track 0.00 -> 391.6 mm, vias 0 -> 9
- net A04: track 0.00 -> 389.1 mm, vias 0 -> 8
- net A08: track 0.00 -> 387.0 mm, vias 0 -> 5
- net A01: track 0.00 -> 384.7 mm, vias 0 -> 9
- net R/W*: track 0.00 -> 383.7 mm, vias 0 -> 3
- net AS*: track 0.00 -> 380.3 mm, vias 0 -> 5
- net A09: track 0.00 -> 324.5 mm, vias 0 -> 5
- net D02: track 0.00 -> 322.1 mm, vias 0 -> 5
- net D05: track 0.00 -> 313.9 mm, vias 0 -> 8
- net A13: track 0.00 -> 313.3 mm, vias 0 -> 5
- net D03: track 0.00 -> 312.5 mm, vias 0 -> 5
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