File: TS2/v2.1/page7.sch (KiCad schematic (older format))
At the start: 11 parts, among them P1 FTDI (TERMINAL), P2 FTDI (HOST), U29 6850, U3 74LS00, U30 6850, U31 MC14411, U5 74LS04, Y1 1.842MHz

Commit message: Rev 2.1 design changes.
Parts:
- removed U31: MC14411, Housings_DIP:DIP-24_W15.24mm, symbol MC14411
- added C39, C40: 22pF, Capacitors_ThroughHole:C_Disc_D3_P2.5, symbol C
- added U31: 74HC4060, Housings_DIP:DIP-16_W7.62mm, symbol 74HC4060
- R20: value 15M -> 10M
- Y1: value 1.842MHz -> 2.4576MHz
Connections:
- net GND: now also C39.1, C40.2, U31.12 (MR), U31.8 (GND)
- net VCC: now also U31.16 (VCC)
- net at U29.3 (RxC), U29.4 (TxC), U30.3 (RxC)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: now also U31.7 (Q4)
- net at R20.1, Y1.2: now also C40.1, U31.10 (~PHI0)
- net at R20.2, Y1.1: now also C39.2, U31.11 (PHI1)
- no-connect marks 9 -> 14
Other:
- moved on the sheet: R20, Y1
Changed lines of the file:
@@
 Sheet 8 9
 Title "TS2 68000 Single Board Computer"
-Date "2017-02-12"
+Date "2017-02-14"
 Rev "2.1"
 Comp "Jeff Tranter"
@@
 $EndComp
 $Comp
-L MC14411 U31
-U 1 1 57C65845
-P 7250 1600
-F 0 "U31" H 7250 1700 50  0000 C CNN
-F 1 "MC14411" H 7250 1500 50  0000 C CNN
-F 2 "Housings_DIP:DIP-24_W15.24mm" H 7250 1600 50  0001 C CNN
-F 3 "" H 7250 1600 50  0000 C CNN
-	1    7250 1600
-	1    0    0    -1
-$EndComp
-$Comp
 L Crystal_Small Y1
 U 1 1 57C66EB0
-P 6350 1850
-F 0 "Y1" H 6350 1950 50  0000 C CNN
-F 1 "1.842MHz" H 6350 1750 50  0000 C CNN
-F 2 "Crystals:Crystal_HC49-U_Vertical" H 6350 1850 50  0001 C CNN
-F 3 "" H 6350 1850 50  0000 C CNN
-	1    6350 1850
+P 6100 1600
+F 0 "Y1" H 6100 1700 50  0000 C CNN
+F 1 "2.4576MHz" H 6100 1500 50  0000 C CNN
+F 2 "Crystals:Crystal_HC49-U_Vertical" H 6100 1600 50  0001 C CNN
+F 3 "" H 6100 1600 50  0000 C CNN
+	1    6100 1600
 	0    1    1    0
 $EndComp
@@
 L R R20
 U 1 1 57C67003
-P 6100 1850
-F 0 "R20" V 6180 1850 50  0000 C CNN
-F 1 "15M" V 6100 1850 50  0000 C CNN
-F 2 "Resistors_ThroughHole:Resistor_Horizontal_RM7mm" V 6030 1850 50  0001 C CNN
-F 3 "" H 6100 1850 50  0000 C CNN
-	1    6100 1850
+P 5850 1600
+F 0 "R20" V 5930 1600 50  0000 C CNN
+F 1 "10M" V 5850 1600 50  0000 C CNN
+F 2 "Resistors_ThroughHole:Resistor_Horizontal_RM7mm" V 5780 1600 50  0001 C CNN
+F 3 "" H 5850 1600 50  0000 C CNN
+	1    5850 1600
 	-1   0    0    1
-$EndComp
-$Comp
-L GND #PWR094
-U 1 1 57C6835F
-P 7250 2050
-F 0 "#PWR094" H 7250 1800 50  0001 C CNN
-F 1 "GND" H 7250 1900 50  0000 C CNN
-F 2 "" H 7250 2050 50  0000 C CNN
-F 3 "" H 7250 2050 50  0000 C CNN
-	1    7250 2050
-	1    0    0    -1
-$EndComp
-$Comp
-L VCC #PWR095
-U 1 1 57C6838D
-P 7250 1150
-F 0 "#PWR095" H 7250 1000 50  0001 C CNN
-F 1 "VCC" H 7250 1300 50  0000 C CNN
-F 2 "" H 7250 1150 50  0000 C CNN
-F 3 "" H 7250 1150 50  0000 C CNN
-	1    7250 1150
-	1    0    0    -1
-$EndComp
-$Comp
-L GND #PWR096
-U 1 1 57C688B5
-P 6450 1450
-F 0 "#PWR096" H 6450 1200 50  0001 C CNN
-F 1 "GND" H 6450 1300 50  0000 C CNN
-F 2 "" H 6450 1450 50  0000 C CNN
-F 3 "" H 6450 1450 50  0000 C CNN
-	1    6450 1450
-	1    0    0    -1
-$EndComp
-$Comp
-L VCC #PWR097
-U 1 1 57C688E3
-P 6450 1250
-F 0 "#PWR097" H 6450 1100 50  0001 C CNN
-F 1 "VCC" H 6450 1400 50  0000 C CNN
-F 2 "" H 6450 1250 50  0000 C CNN
-F 3 "" H 6450 1250 50  0000 C CNN
-	1    6450 1250
-	1    0    0    -1
 $EndComp
 Text GLabel 2050 1750 0    60   Input ~ 0
@@
 D15
 $Comp
-L VCC #PWR098
+L VCC #PWR093
 U 1 1 57C7A398
 P 3800 1650
-F 0 "#PWR098" H 3800 1500 50  0001 C CNN
+F 0 "#PWR093" H 3800 1500 50  0001 C CNN
 F 1 "VCC" H 3800 1800 50  0000 C CNN
 F 2 "" H 3800 1650 50  0000 C CNN
@@
 $EndComp
 $Comp
-L GND #PWR099
+L GND #PWR094
 U 1 1 57C7A4BC
 P 3800 3550
-F 0 "#PWR099" H 3800 3300 50  0001 C CNN
+F 0 "#PWR094" H 3800 3300 50  0001 C CNN
 F 1 "GND" H 3800 3400 50  0000 C CNN
 F 2 "" H 3800 3550 50  0000 C CNN
@@
 $EndComp
 $Comp
-L VCC #PWR0100
+L VCC #PWR095
 U 1 1 57C7A5E0
 P 3800 4500
-F 0 "#PWR0100" H 3800 4350 50  0001 C CNN
+F 0 "#PWR095" H 3800 4350 50  0001 C CNN
 F 1 "VCC" H 3800 4650 50  0000 C CNN
 F 2 "" H 3800 4500 50  0000 C CNN
@@
 $EndComp
 $Comp
-L GND #PWR0101
+L GND #PWR096
 U 1 1 57C7A616
 P 3800 6400
-F 0 "#PWR0101" H 3800 6150 50  0001 C CNN
+F 0 "#PWR096" H 3800 6150 50  0001 C CNN
 F 1 "GND" H 3800 6250 50  0000 C CNN
 F 2 "" H 3800 6400 50  0000 C CNN
@@
 	1    0    0    -1
 $EndComp
-NoConn ~ 8050 1350
-NoConn ~ 8050 1450
-NoConn ~ 8050 1550
-NoConn ~ 8050 1650
-NoConn ~ 8050 1750
+NoConn ~ 7800 1100
+NoConn ~ 7800 1200
+NoConn ~ 7800 1300
+NoConn ~ 7800 1400
+NoConn ~ 7800 1500
 $Comp
 L CONN_01X06 P1
@@
 $EndComp
 $Comp
-L GND #PWR0102
+L GND #PWR097
 U 1 1 57CB2088
 P 8450 2000
-F 0 "#PWR0102" H 8450 1750 50  0001 C CNN
+F 0 "#PWR097" H 8450 1750 50  0001 C CNN
 F 1 "GND" H 8450 1850 50  0000 C CNN
 F 2 "" H 8450 2000 50  0000 C CNN
@@
 $EndComp
 $Comp
-L GND #PWR0103
+L GND #PWR098
 U 1 1 57CB2D6B
 P 4500 3000
-F 0 "#PWR0103" H 4500 2750 50  0001 C CNN
+F 0 "#PWR098" H 4500 2750 50  0001 C CNN
 F 1 "GND" H 4500 2850 50  0000 C CNN
 F 2 "" H 4500 3000 50  0000 C CNN
@@
 $EndComp
 $Comp
-L GND #PWR0104
+L GND #PWR099
 U 1 1 57CB394C
 P 8450 4850
-F 0 "#PWR0104" H 8450 4600 50  0001 C CNN
+F 0 "#PWR099" H 8450 4600 50  0001 C CNN
 F 1 "GND" H 8450 4700 50  0000 C CNN
 F 2 "" H 8450 4850 50  0000 C CNN
@@
 $EndComp
 $Comp
-L GND #PWR0105
+L GND #PWR0100
 U 1 1 57CB4274
 P 4500 5850
-F 0 "#PWR0105" H 4500 5600 50  0001 C CNN
+F 0 "#PWR0100" H 4500 5600 50  0001 C CNN
 F 1 "GND" H 4500 5700 50  0000 C CNN
 F 2 "" H 4500 5850 50  0000 C CNN
@@
 NoConn ~ 8600 5350
 NoConn ~ 8600 4950
-Text Notes 8300 1300 0    60   ~ 0
+Text Notes 8300 1050 0    60   ~ 0
 9600
-Text Notes 8300 1400 0    60   ~ 0
+Text Notes 8300 1150 0    60   ~ 0
 4800
-Text Notes 8300 1500 0    60   ~ 0
+Text Notes 8300 1250 0    60   ~ 0
 2400
-Text Notes 8300 1600 0    60   ~ 0
+Text Notes 8300 1350 0    60   ~ 0
 1200
-Text Notes 8300 1700 0    60   ~ 0
+Text Notes 8350 1450 0    60   ~ 0
 600
-Text Notes 8300 1800 0    60   ~ 0
+Text Notes 8350 1550 0    60   ~ 0
 300
-Text Notes 8600 1550 0    60   ~ 0
+Text Notes 8650 1350 0    60   ~ 0
 Select baud rate (console and aux.\nports can use different baud rates\nif desired).
 Wire Wire Line
-	6100 1700 6450 1700
-Wire Wire Line
-	6100 2000 6450 2000
-Wire Wire Line
-	6350 1950 6350 2000
-Connection ~ 6350 2000
-Wire Wire Line
-	6350 1750 6350 1700
-Connection ~ 6350 1700
-Wire Wire Line
-	6450 1250 6450 1350
-Wire Wire Line
 	3100 1750 2050 1750
-Wire Wire Line
-	8050 1250 8200 1250
-Wire Wire Line
-	8050 1250 8050 800
 Wire Wire Line
 	4500 1850 4500 1750
@@
 	5100 4700 4500 4700
 Wire Wire Line
-	4500 1850 5300 1850
+	4500 1850 5200 1850
 Connection ~ 4500 4700
 Wire Wire Line
 	4500 4700 4500 4600
 Wire Wire Line
-	8050 800  5300 800
+	8050 700  5200 700
 Text Notes 9450 2250 0    60   ~ 0
 FTDI (USB to\nserial adaptor)
@@
 NoConn ~ 8600 2100
 Wire Wire Line
-	5300 800  5300 1850
+	5200 700  5200 1850
 Wire Wire Line
 	5100 4700 5100 600
 Wire Wire Line
 	5100 600  8200 600
-Wire Wire Line
-	8200 600  8200 1250
-Connection ~ 8050 1250
 $Comp
 L Jumper_NO_Small JP5
@@
 Text GLabel 8100 5050 0    60   Output ~ 0
 POWER
+$Comp
+L 74HC4060 U31
+U 1 1 58A0CD07
+P 7100 1500
+F 0 "U31" H 7100 1600 50  0000 C CNN
+F 1 "74HC4060" H 7100 1350 50  0000 C CNN
+F 2 "Housings_DIP:DIP-16_W7.62mm" H 7100 1500 50  0001 C CNN
+F 3 "" H 7100 1500 50  0000 C CNN
+	1    7100 1500
+	1    0    0    -1
+$EndComp
+Wire Wire Line
+	5850 1400 6400 1400
+Wire Wire Line
+	5850 1400 5850 1450
+Wire Wire Line
+	6100 1500 6100 1400
+Connection ~ 6100 1400
+Wire Wire Line
+	5850 1750 5850 1800
+Wire Wire Line
+	5850 1800 6400 1800
+Wire Wire Line
+	6100 1700 6100 1800
+Connection ~ 6100 1800
+$Comp
+L GND #PWR0101
+U 1 1 58A0DB54
+P 7100 2050
+F 0 "#PWR0101" H 7100 1800 50  0001 C CNN
+F 1 "GND" H 7100 1900 50  0000 C CNN
+F 2 "" H 7100 2050 50  0000 C CNN
+F 3 "" H 7100 2050 50  0000 C CNN
+	1    7100 2050
+	1    0    0    -1
+$EndComp
+$Comp
+L VCC #PWR0102
+U 1 1 58A0DBF7
+P 7100 950
+F 0 "#PWR0102" H 7100 800 50  0001 C CNN
+F 1 "VCC" H 7100 1100 50  0000 C CNN
+F 2 "" H 7100 950 50  0000 C CNN
+F 3 "" H 7100 950 50  0000 C CNN
+	1    7100 950
+	1    0    0    -1
+$EndComp
+Wire Wire Line
+	7800 1000 8200 1000
+Wire Wire Line
+	8050 1000 8050 700
+Wire Wire Line
+	8200 1000 8200 600
+Connection ~ 8050 1000
+NoConn ~ 7800 1600
+NoConn ~ 7800 1700
+NoConn ~ 7800 1800
+NoConn ~ 7800 1900
+$Comp
+L GND #PWR0103
+U 1 1 58A0F2FA
+P 6400 1100
+F 0 "#PWR0103" H 6400 850 50  0001 C CNN
+F 1 "GND" H 6400 950 50  0000 C CNN
+F 2 "" H 6400 1100 50  0000 C CNN
+F 3 "" H 6400 1100 50  0000 C CNN
+	1    6400 1100
+	1    0    0    -1
+$EndComp
+NoConn ~ 6400 1600
+$Comp
+L C C40
+U 1 1 58A1071E
+P 6100 1950
+F 0 "C40" H 6125 2050 50  0000 L CNN
+F 1 "22pF" H 6125 1850 50  0000 L CNN
+F 2 "Capacitors_ThroughHole:C_Disc_D3_P2.5" H 6138 1800 50  0001 C CNN
+F 3 "" H 6100 1950 50  0000 C CNN
+	1    6100 1950
+	1    0    0    -1
+$EndComp
+$Comp
+L GND #PWR0104
+U 1 1 58A10767
+P 6100 2100
+F 0 "#PWR0104" H 6100 1850 50  0001 C CNN
+F 1 "GND" H 6100 1950 50  0000 C CNN
+F 2 "" H 6100 2100 50  0000 C CNN
+F 3 "" H 6100 2100 50  0000 C CNN
+	1    6100 2100
+	1    0    0    -1
+$EndComp
+$Comp
+L C C39
+U 1 1 58A10795
+P 6100 1250
+F 0 "C39" H 6125 1350 50  0000 L CNN
+F 1 "22pF" H 6125 1150 50  0000 L CNN
+F 2 "Capacitors_ThroughHole:C_Disc_D3_P2.5" H 6138 1100 50  0001 C CNN
+F 3 "" H 6100 1250 50  0000 C CNN
+	1    6100 1250
+	1    0    0    -1
+$EndComp
+$Comp
+L GND #PWR0105
+U 1 1 58A107D4
+P 6100 1100
+F 0 "#PWR0105" H 6100 850 50  0001 C CNN
+F 1 "GND" H 6100 950 50  0000 C CNN
+F 2 "" H 6100 1100 50  0000 C CNN
+F 3 "" H 6100 1100 50  0000 C CNN
+	1    6100 1100
+	-1   0    0    1
+$EndComp
 $EndSCHEMATC
