File: TS2/v2.1/ts2.sch (KiCad schematic (older format))
At the start: 43 parts, among them P3 +5V POWER, SW5 POWER, U10 74LS32, U34 74LS00, U35 74LS74

Commit message: Rev 2.1 design changes.
Parts:
- removed U34: 74LS00, Housings_DIP:DIP-14_W7.62mm, symbol 74LS00
- added C41, C42: 0.1uF, Capacitors_ThroughHole:C_Disc_D3_P2.5, symbol C
- added U36: 74LS27, Housings_DIP:DIP-14_W7.62mm, symbol 74LS27
Connections:
- net GND: now also C41.2, C42.2, U36.10, U36.11, U36.3, U36.4, U36.5, U36.7 (GND), U36.7 (GND), U36.9
- net VCC: now also C41.1, C42.1, U36.14 (VCC), U36.14 (VCC)
- no-connect marks 4 -> 5
Changed lines of the file:
@@
 Sheet 1 9
 Title "TS2 68000 Single Board Computer"
-Date "2017-02-14"
+Date "2017-02-15"
 Rev "2.1"
 Comp "Jeff Tranter"
@@
 $EndComp
 $Comp
-L 74LS00 U34
-U 4 1 587B2C0E
-P 5900 5300
-F 0 "U34" H 5900 5350 50  0000 C CNN
-F 1 "74LS00" H 5900 5200 50  0000 C CNN
-F 2 "Housings_DIP:DIP-14_W7.62mm" H 5900 5300 50  0001 C CNN
-F 3 "" H 5900 5300 50  0000 C CNN
-	4    5900 5300
-	1    0    0    -1
-$EndComp
-$Comp
 L 74LS74 U35
 U 2 1 587B2C8B
@@
 $Comp
 L GND #PWR015
-U 1 1 587B30E5
-P 5300 5400
-F 0 "#PWR015" H 5300 5150 50  0001 C CNN
-F 1 "GND" H 5300 5250 50  0000 C CNN
-F 2 "" H 5300 5400 50  0000 C CNN
-F 3 "" H 5300 5400 50  0000 C CNN
-	1    5300 5400
-	1    0    0    -1
-$EndComp
-$Comp
-L GND #PWR016
-U 1 1 587B3109
-P 5300 5200
-F 0 "#PWR016" H 5300 4950 50  0001 C CNN
-F 1 "GND" H 5300 5050 50  0000 C CNN
-F 2 "" H 5300 5200 50  0000 C CNN
-F 3 "" H 5300 5200 50  0000 C CNN
-	1    5300 5200
-	1    0    0    -1
-$EndComp
-NoConn ~ 6500 5300
-$Comp
-L GND #PWR017
 U 1 1 587B3523
 P 6750 4800
-F 0 "#PWR017" H 6750 4550 50  0001 C CNN
+F 0 "#PWR015" H 6750 4550 50  0001 C CNN
 F 1 "GND" H 6750 4650 50  0000 C CNN
 F 2 "" H 6750 4800 50  0000 C CNN
@@
 $EndComp
 $Comp
-L GND #PWR018
+L GND #PWR016
 U 1 1 587B3547
 P 6750 5000
-F 0 "#PWR018" H 6750 4750 50  0001 C CNN
+F 0 "#PWR016" H 6750 4750 50  0001 C CNN
 F 1 "GND" H 6750 4850 50  0000 C CNN
 F 2 "" H 6750 5000 50  0000 C CNN
@@
 $EndComp
 $Comp
-L GND #PWR019
+L GND #PWR017
 U 1 1 587B356B
 P 7350 5550
-F 0 "#PWR019" H 7350 5300 50  0001 C CNN
+F 0 "#PWR017" H 7350 5300 50  0001 C CNN
 F 1 "GND" H 7350 5400 50  0000 C CNN
 F 2 "" H 7350 5550 50  0000 C CNN
@@
 $EndComp
 $Comp
-L GND #PWR020
+L GND #PWR018
 U 1 1 587B358F
 P 7350 4450
-F 0 "#PWR020" H 7350 4200 50  0001 C CNN
+F 0 "#PWR018" H 7350 4200 50  0001 C CNN
 F 1 "GND" H 7350 4300 50  0000 C CNN
 F 2 "" H 7350 4450 50  0000 C CNN
@@
 $EndComp
 $Comp
-L VCC #PWR021
+L VCC #PWR019
 U 1 1 587B86B5
 P 3150 5450
-F 0 "#PWR021" H 3150 5300 50  0001 C CNN
+F 0 "#PWR019" H 3150 5300 50  0001 C CNN
 F 1 "VCC" H 3150 5600 50  0000 C CNN
 F 2 "" H 3150 5450 50  0000 C CNN
@@
 $EndComp
 $Comp
-L GND #PWR022
+L GND #PWR020
 U 1 1 587B86DD
 P 2150 5550
-F 0 "#PWR022" H 2150 5300 50  0001 C CNN
+F 0 "#PWR020" H 2150 5300 50  0001 C CNN
 F 1 "GND" H 2150 5400 50  0000 C CNN
 F 2 "" H 2150 5550 50  0000 C CNN
@@
 $EndComp
 $Comp
-L GND #PWR023
+L GND #PWR021
 U 1 1 588696BC
 P 1850 7250
-F 0 "#PWR023" H 1850 7000 50  0001 C CNN
+F 0 "#PWR021" H 1850 7000 50  0001 C CNN
 F 1 "GND" H 1850 7100 50  0000 C CNN
 F 2 "" H 1850 7250 50  0000 C CNN
@@
 $EndComp
 $Comp
-L VCC #PWR024
+L VCC #PWR022
 U 1 1 588696C2
 P 1850 6950
-F 0 "#PWR024" H 1850 6800 50  0001 C CNN
+F 0 "#PWR022" H 1850 6800 50  0001 C CNN
 F 1 "VCC" H 1850 7100 50  0000 C CNN
 F 2 "" H 1850 6950 50  0000 C CNN
@@
 $EndComp
 $Comp
-L GND #PWR025
+L GND #PWR023
 U 1 1 5886A465
 P 5000 7250
-F 0 "#PWR025" H 5000 7000 50  0001 C CNN
+F 0 "#PWR023" H 5000 7000 50  0001 C CNN
 F 1 "GND" H 5000 7100 50  0000 C CNN
 F 2 "" H 5000 7250 50  0000 C CNN
@@
 $EndComp
 $Comp
-L VCC #PWR026
+L VCC #PWR024
 U 1 1 5886A46B
 P 5000 6950
-F 0 "#PWR026" H 5000 6800 50  0001 C CNN
+F 0 "#PWR024" H 5000 6800 50  0001 C CNN
 F 1 "VCC" H 5000 7100 50  0000 C CNN
 F 2 "" H 5000 6950 50  0000 C CNN
@@
 $EndComp
 $Comp
-L GND #PWR027
+L GND #PWR025
 U 1 1 5886CFC8
 P 5000 6500
-F 0 "#PWR027" H 5000 6250 50  0001 C CNN
+F 0 "#PWR025" H 5000 6250 50  0001 C CNN
 F 1 "GND" H 5000 6350 50  0000 C CNN
 F 2 "" H 5000 6500 50  0000 C CNN
@@
 $EndComp
 $Comp
-L VCC #PWR028
+L VCC #PWR026
 U 1 1 5886CFCE
 P 5000 6200
-F 0 "#PWR028" H 5000 6050 50  0001 C CNN
+F 0 "#PWR026" H 5000 6050 50  0001 C CNN
 F 1 "VCC" H 5000 6350 50  0000 C CNN
 F 2 "" H 5000 6200 50  0000 C CNN
@@
 	1    0    0    -1
 $EndComp
-Wire Wire Line
-	5000 6200 7700 6200
 Connection ~ 7400 6200
 Connection ~ 7100 6200
@@
 Connection ~ 5600 6200
 Connection ~ 5300 6200
-Wire Wire Line
-	5000 6500 7700 6500
 Connection ~ 7400 6500
 Connection ~ 7100 6500
@@
 Connection ~ 5000 6200
 Connection ~ 5000 6500
+$Comp
+L 74LS27 U36
+U 2 1 58A4EF34
+P 9300 4550
+F 0 "U36" H 9300 4600 50  0000 C CNN
+F 1 "74LS27" H 9300 4500 50  0000 C CNN
+F 2 "Housings_DIP:DIP-14_W7.62mm" H 9300 4550 50  0001 C CNN
+F 3 "" H 9300 4550 50  0000 C CNN
+	2    9300 4550
+	1    0    0    -1
+$EndComp
+$Comp
+L 74LS27 U36
+U 3 1 58A4F156
+P 9300 5600
+F 0 "U36" H 9300 5650 50  0000 C CNN
+F 1 "74LS27" H 9300 5550 50  0000 C CNN
+F 2 "Housings_DIP:DIP-14_W7.62mm" H 9300 5600 50  0001 C CNN
+F 3 "" H 9300 5600 50  0000 C CNN
+	3    9300 5600
+	1    0    0    -1
+$EndComp
+NoConn ~ 9900 5600
+NoConn ~ 9900 4550
+$Comp
+L GND #PWR027
+U 1 1 58A5213C
+P 8700 5450
+F 0 "#PWR027" H 8700 5200 50  0001 C CNN
+F 1 "GND" H 8700 5300 50  0000 C CNN
+F 2 "" H 8700 5450 50  0000 C CNN
+F 3 "" H 8700 5450 50  0000 C CNN
+	1    8700 5450
+	1    0    0    -1
+$EndComp
+$Comp
+L GND #PWR028
+U 1 1 58A521B4
+P 8700 5600
+F 0 "#PWR028" H 8700 5350 50  0001 C CNN
+F 1 "GND" H 8700 5450 50  0000 C CNN
+F 2 "" H 8700 5600 50  0000 C CNN
+F 3 "" H 8700 5600 50  0000 C CNN
+	1    8700 5600
+	1    0    0    -1
+$EndComp
+$Comp
+L GND #PWR029
+U 1 1 58A5222C
+P 8700 5750
+F 0 "#PWR029" H 8700 5500 50  0001 C CNN
+F 1 "GND" H 8700 5600 50  0000 C CNN
+F 2 "" H 8700 5750 50  0000 C CNN
+F 3 "" H 8700 5750 50  0000 C CNN
+	1    8700 5750
+	1    0    0    -1
+$EndComp
+$Comp
+L GND #PWR030
+U 1 1 58A522A4
+P 8700 4400
+F 0 "#PWR030" H 8700 4150 50  0001 C CNN
+F 1 "GND" H 8700 4250 50  0000 C CNN
+F 2 "" H 8700 4400 50  0000 C CNN
+F 3 "" H 8700 4400 50  0000 C CNN
+	1    8700 4400
+	1    0    0    -1
+$EndComp
+$Comp
+L GND #PWR031
+U 1 1 58A5231C
+P 8700 4550
+F 0 "#PWR031" H 8700 4300 50  0001 C CNN
+F 1 "GND" H 8700 4400 50  0000 C CNN
+F 2 "" H 8700 4550 50  0000 C CNN
+F 3 "" H 8700 4550 50  0000 C CNN
+	1    8700 4550
+	1    0    0    -1
+$EndComp
+$Comp
+L GND #PWR032
+U 1 1 58A52394
+P 8700 4700
+F 0 "#PWR032" H 8700 4450 50  0001 C CNN
+F 1 "GND" H 8700 4550 50  0000 C CNN
+F 2 "" H 8700 4700 50  0000 C CNN
+F 3 "" H 8700 4700 50  0000 C CNN
+	1    8700 4700
+	1    0    0    -1
+$EndComp
+$Comp
+L C C41
+U 1 1 58A53932
+P 8000 6350
+F 0 "C41" H 8025 6450 50  0000 L CNN
+F 1 "0.1uF" H 8025 6250 50  0000 L CNN
+F 2 "Capacitors_ThroughHole:C_Disc_D3_P2.5" H 8038 6200 50  0001 C CNN
+F 3 "" H 8000 6350 50  0000 C CNN
+	1    8000 6350
+	1    0    0    -1
+$EndComp
+$Comp
+L C C42
+U 1 1 58A53A21
+P 8300 6350
+F 0 "C42" H 8325 6450 50  0000 L CNN
+F 1 "0.1uF" H 8325 6250 50  0000 L CNN
+F 2 "Capacitors_ThroughHole:C_Disc_D3_P2.5" H 8338 6200 50  0001 C CNN
+F 3 "" H 8300 6350 50  0000 C CNN
+	1    8300 6350
+	1    0    0    -1
+$EndComp
+Connection ~ 7700 6200
+Connection ~ 8000 6200
+Connection ~ 8300 6200
+Connection ~ 7700 6500
+Connection ~ 8000 6500
+Connection ~ 8300 6500
+Wire Wire Line
+	5000 6200 8300 6200
+Wire Wire Line
+	8300 6500 5000 6500
 $EndSCHEMATC

Commit message: Rev 2.1.1 changes.
Connections:
- net POWER: now also P3.2 (P2), SW5.1
Other:
- moved on the sheet: SW5
Changed lines of the file:
@@
 Sheet 1 9
 Title "TS2 68000 Single Board Computer"
-Date "2017-02-17"
-Rev "2.1"
+Date "2017-05-29"
+Rev "2.1.1"
 Comp "Jeff Tranter"
 Comment1 "Top Level Schematic"
@@
 L SPST SW5
 U 1 1 587B85F6
-P 2650 5450
-F 0 "SW5" H 2650 5550 50  0000 C CNN
-F 1 "POWER" H 2650 5350 50  0000 C CNN
-F 2 "Connect:PINHEAD1-3" H 2650 5450 50  0001 C CNN
-F 3 "" H 2650 5450 50  0000 C CNN
-	1    2650 5450
+P 2850 5450
+F 0 "SW5" H 2850 5550 50  0000 C CNN
+F 1 "POWER" H 2850 5350 50  0000 C CNN
+F 2 "Connect:PINHEAD1-3" H 2850 5450 50  0001 C CNN
+F 3 "" H 2850 5450 50  0000 C CNN
+	1    2850 5450
 	1    0    0    -1
 $EndComp
@@
 L VCC #PWR019
 U 1 1 587B86B5
-P 3150 5450
-F 0 "#PWR019" H 3150 5300 50  0001 C CNN
-F 1 "VCC" H 3150 5600 50  0000 C CNN
-F 2 "" H 3150 5450 50  0000 C CNN
-F 3 "" H 3150 5450 50  0000 C CNN
-	1    3150 5450
+P 3350 5450
+F 0 "#PWR019" H 3350 5300 50  0001 C CNN
+F 1 "VCC" H 3350 5600 50  0000 C CNN
+F 2 "" H 3350 5450 50  0000 C CNN
+F 3 "" H 3350 5450 50  0000 C CNN
+	1    3350 5450
 	1    0    0    -1
 $EndComp
@@
 	1    0    0    -1
 $EndComp
-Text GLabel 2550 6000 2    60   Input ~ 0
+Text GLabel 2500 5850 2    60   Input ~ 0
 POWER
-Wire Wire Line
-	2550 6000 2250 6000
-Wire Wire Line
-	2250 6000 2250 5450
-Connection ~ 2250 5450
 $Comp
 L C C6
@@
 Wire Wire Line
 	8300 6500 5000 6500
+Wire Wire Line
+	2150 5450 2350 5450
+Wire Wire Line
+	2300 5850 2300 5450
+Connection ~ 2300 5450
+Wire Wire Line
+	2500 5850 2300 5850
 $EndSCHEMATC
